Commit message: mitsubishi arm hardware interface new tests...

File: barrett_hand_description/robots/bhand_model.URDF (robot description, URDF)
Before this commit: robot barret_hand_description, 9 links, 8 joints
Links:
- removed link barret_base_link
- added link barrett_base_link, mass 0.377966381303299; collision mesh filename=package://barrett_hand_description/meshes/base_link.STL; visual mesh filename=package://barrett_hand_description/meshes/base_link.STL
- link finger_1_dist_link: geometry collision mesh filename=package://barrett_hand_description/meshes/finger_1_dist_lin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; visual mesh filename=package://barrett_hand_description/meshes/finger_1_dist_lin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
- link finger_1_med_liink: geometry collision mesh filename=package://barrett_hand_description/meshes/finger_1_med_liin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; visual mesh filename=package://barrett_hand_description/meshes/finger_1_med_liin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
- link finger_1_prox_link: geometry collision mesh filename=package://barrett_hand_description/meshes/finger_1_prox_lin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; visual mesh filename=package://barrett_hand_description/meshes/finger_1_prox_lin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
- link finger_2_dist_link: geometry collision mesh filename=package://barrett_hand_description/meshes/finger_2_dist_lin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; visual mesh filename=package://barrett_hand_description/meshes/finger_2_dist_lin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
- link finger_2_med_link: geometry collision mesh filename=package://barrett_hand_description/meshes/finger_2_med_link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; visual mesh filename=package://barrett_hand_description/meshes/finger_2_med_link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
- link finger_2_prox_link: geometry collision mesh filename=package://barrett_hand_description/meshes/finger_2_prox_lin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; visual mesh filename=package://barrett_hand_description/meshes/finger_2_prox_lin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
- link finger_3_dist_link: geometry collision mesh filename=package://barrett_hand_description/meshes/finger_3_dist_lin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; visual mesh filename=package://barrett_hand_description/meshes/finger_3_dist_lin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
- link finger_3_med_link: geometry collision mesh filename=package://barrett_hand_description/meshes/finger_3_med_link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; visual mesh filename=package://barrett_hand_description/meshes/finger_3_med_link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
Joints:
- joint finger_1_prox_joint: parent barret_base_link -> barrett_base_link
- joint finger_2_prox_joint: parent barret_base_link -> barrett_base_link
- joint finger_3_med_joint: parent barret_base_link -> barrett_base_link
