Commit message: barrett hand position hardware interface and controllers implemented

File: barrett_hand_description/urdf/barrett_hand.xacro (robot description, xacro)
@@ -1,6 +1,5 @@
-<robot
-  name="barrett_hand_description">
-  <link
-    name="barrett_base_link">
+<?xml version="1.0"?>
+<robot xmlns:xacro="http://www.ros.org/wiki/xacro">
+  <link name="barrett_base_link">
     <inertial>
       <origin
@@ -84,11 +83,11 @@
       xyz="0 0 1" />
     <limit
-      lower="-3.141"
-      upper="0"
-      effort="0"
-      velocity="0" />
-  </joint>
-  <link
-    name="finger_1_med_liink">
+      lower="0.0"
+      upper="3.141"
+      effort="0"
+      velocity="0" />
+  </joint>
+  <link
+    name="finger_1_med_link">
     <inertial>
       <origin
@@ -111,5 +110,5 @@
       <geometry>
         <mesh
-          filename="package://barrett_hand_description/meshes/finger_1_med_liink.STL" />
+          filename="package://barrett_hand_description/meshes/finger_1_med_link.STL" />
       </geometry>
       <material
@@ -125,5 +124,5 @@
       <geometry>
         <mesh
-          filename="package://barrett_hand_description/meshes/finger_1_med_liink.STL" />
+          filename="package://barrett_hand_description/meshes/finger_1_med_link.STL" />
       </geometry>
     </collision>
@@ -134,14 +133,14 @@
     <origin
       xyz="-0.05 0 0.0339"
-      rpy="1.5708 -8.8281E-17 0" />
+      rpy="-1.5708 -8.8281E-17 0" />
     <parent
       link="finger_1_prox_link" />
     <child
-      link="finger_1_med_liink" />
-    <axis
-      xyz="0 0 1" />
-    <limit
-      lower="-2.44"
-      upper="0"
+      link="finger_1_med_link" />
+    <axis
+      xyz="0 0 1" />
+    <limit
+      lower="0"
+      upper="2.44"
       effort="0"
       velocity="0" />
@@ -189,10 +188,10 @@
   <joint
     name="finger_1_dist_joint"
-    type="revolute">
+    type="fixed"> <!--original is revolute-->
     <origin
       xyz="-0.069936 0.003 0"
       rpy="1.6787E-18 -3.6382E-15 -6.1073E-33" />
     <parent
-      link="finger_1_med_liink" />
+      link="finger_1_med_link" />
     <child
       link="finger_1_dist_link" />
@@ -308,5 +307,5 @@
     <origin
       xyz="-0.05 0 0.0339"
-      rpy="1.5708 -8.8281E-17 0" />
+      rpy="-1.5708 -8.8281E-17 0" />
     <parent
       link="finger_2_prox_link" />
@@ -316,6 +315,6 @@
       xyz="0 0 1" />
     <limit
-      lower="-2.44"
-      upper="0"
+      lower="0.0"
+      upper="2.44"
       effort="0"
       velocity="0" />
@@ -363,5 +362,5 @@
   <joint
     name="finger_2_dist_joint"
-    type="revolute">
+    type="fixed"> <!--original is revolute-->
     <origin
       xyz="-0.069917 0.0034087 0"
@@ -424,5 +423,5 @@
     <origin
       xyz="0 -0.05 0.0754"
-      rpy="1.5708 6.123E-17 1.5708" />
+      rpy="-1.5708 6.123E-17 1.5708" />
     <parent
       link="barrett_base_link" />
@@ -432,6 +431,6 @@
       xyz="0 0 1" />
     <limit
-      lower="-2.44"
-      upper="0"
+      lower="0.0"
+      upper="2.44"
       effort="0"
       velocity="0" />
@@ -479,5 +478,5 @@
   <joint
     name="finger_3_dist_joint"
-    type="revolute">
+    type="fixed"> <!--original is revolute-->
     <origin
       xyz="-0.069936 0.003 0"

Commit message: barrett hand moveit planner is working

File: barrett_hand_description/urdf/barrett_hand.xacro (robot description, xacro)
@@ -2,5 +2,5 @@
 <robot xmlns:xacro="http://www.ros.org/wiki/xacro">
   <link name="barrett_base_link">
-    <inertial>
+    <!--<inertial>
       <origin
         xyz="-1.53444878605399E-05 -0.00277693660903533 0.0352882290973172"
@@ -15,5 +15,5 @@
         iyz="-3.0792687327603E-05"
         izz="0.000376798128588446" />
-    </inertial>
+    </inertial>-->
     <visual>
       <origin
@@ -81,5 +81,5 @@
       link="finger_1_prox_link" />
     <axis
-      xyz="0 0 1" />
+      xyz="0 0 -1" />
     <limit
       lower="0.0"
@@ -107,5 +107,5 @@
       <origin
         xyz="0 0 0"
-        rpy="0 0 0" />
+        rpy="3.14159265359 0 0" />
       <geometry>
         <mesh
@@ -165,5 +165,5 @@
       <origin
         xyz="0 0 0"
-        rpy="0 0 0" />
+        rpy="3.14159265359 0 0" />
       <geometry>
         <mesh
@@ -190,5 +190,5 @@
     type="fixed"> <!--original is revolute-->
     <origin
-      xyz="-0.069936 0.003 0"
+      xyz="-0.069936 -0.003 0"
       rpy="1.6787E-18 -3.6382E-15 -6.1073E-33" />
     <parent
@@ -199,6 +199,6 @@
       xyz="0 0 1" />
     <limit
-      lower="-0.785"
-      upper="0"
+      lower="0"
+      upper="0.785"
       effort="0"
       velocity="0" />
@@ -281,5 +281,5 @@
       <origin
         xyz="0 0 0"
-        rpy="0 0 0" />
+        rpy="3.14159265359 0 0" />
       <geometry>
         <mesh
@@ -339,5 +339,5 @@
       <origin
         xyz="0 0 0"
-        rpy="0 0 0" />
+        rpy="3.14159265359 0 0" />
       <geometry>
         <mesh
@@ -364,5 +364,5 @@
     type="fixed"> <!--original is revolute-->
     <origin
-      xyz="-0.069917 0.0034087 0"
+      xyz="-0.069917 -0.0034087 0"
       rpy="-3.1382E-17 -2.3229E-16 0" />
     <parent
@@ -397,5 +397,5 @@
       <origin
         xyz="0 0 0"
-        rpy="0 0 0" />
+        rpy="3.14159265359 0 0" />
       <geometry>
         <mesh
@@ -455,5 +455,5 @@
       <origin
         xyz="0 0 0"
-        rpy="0 0 0" />
+        rpy="3.14159265359 0 0" />
       <geometry>
         <mesh
@@ -480,5 +480,5 @@
     type="fixed"> <!--original is revolute-->
     <origin
-      xyz="-0.069936 0.003 0"
+      xyz="-0.069936 -0.003 0"
       rpy="6.0427E-17 -6.7283E-18 -4.0657E-34" />
     <parent

Commit message: updated barrett and mitsubishi arm files for the gazebo simulator

File: barrett_hand_description/urdf/barrett_hand.xacro (robot description, xacro)
@@ -3,10 +3,7 @@
   <link name="barrett_base_link">
     <inertial>
-      <origin xyz="0 0 1" rpy="0 0 0"/>
-      <mass value="0.0001"/>
-      <inertia
-        ixx="1.0" ixy="0.0" ixz="0.0"
-        iyy="1.0" iyz="0.0"
-        izz="1.0"/>
+      <mass value="0.1" />
+      <origin xyz="0 0 0" rpy="0 0 0"/>
+      <inertia ixx="1" ixy="0" ixz="0" iyy="1" iyz="0" izz="1" />
     </inertial>
     <visual>
@@ -30,10 +27,7 @@
   <link name="finger_1_prox_link">
     <inertial>
-      <origin xyz="0 0 1" rpy="0 0 0"/>
-      <mass value="0.0001"/>
-      <inertia
-        ixx="1.0" ixy="0.0" ixz="0.0"
-        iyy="1.0" iyz="0.0"
-        izz="1.0"/>
+      <mass value="0.1" />
+      <origin xyz="0 0 0" rpy="0 0 0"/>
+      <inertia ixx="1" ixy="0" ixz="0" iyy="1" iyz="0" izz="1" />
     </inertial>
     <visual>
@@ -76,17 +70,14 @@
       lower="0.0"
       upper="3.141"
-      effort="0"
-      velocity="0.01" />
-   <dynamics damping="0.0" friction="0.0" />
+      effort="10000"
+      velocity="0.01" />
+   <dynamics damping="10.0" friction="10.0" />
   </joint>
   <link
     name="finger_1_med_link">
     <inertial>
-      <origin xyz="0 0 1" rpy="0 0 0"/>
-      <mass value="0.0001"/>
-      <inertia
-        ixx="1.0" ixy="0.0" ixz="0.0"
-        iyy="1.0" iyz="0.0"
-        izz="1.0"/>
+      <mass value="0.1" />
+      <origin xyz="0 0 0" rpy="0 0 0"/>
+      <inertia ixx="1" ixy="0" ixz="0" iyy="1" iyz="0" izz="1" />
     </inertial>
     <visual>
@@ -129,17 +120,14 @@
       lower="0"
       upper="2.44"
-      effort="0"
-      velocity="0.01" />
-   <dynamics damping="0.0" friction="0.0" />
+      effort="10000"
+      velocity="0.01" />
+   <dynamics damping="10.0" friction="10.0" />
   </joint>
   <link
     name="finger_1_dist_link">
     <inertial>
-      <origin xyz="0 0 1" rpy="0 0 0"/>
-      <mass value="0.0001"/>
-      <inertia
-        ixx="1.0" ixy="0.0" ixz="0.0"
-        iyy="1.0" iyz="0.0"
-        izz="1.0"/>
+      <mass value="0.001" />
+      <origin xyz="0 0 0" rpy="0 0 0"/>
+      <inertia ixx="1" ixy="0" ixz="0" iyy="1" iyz="0" izz="1" />
     </inertial>
     <visual>
@@ -182,17 +170,14 @@
       lower="0.6"
       upper="1.57"
-      effort="0"
-      velocity="0.01" />
-   <dynamics damping="0.0" friction="0.0" />
+      effort="10000"
+      velocity="0.01" />
+   <dynamics damping="10.0" friction="10.0" />
   </joint>
   <link
     name="finger_2_prox_link">
     <inertial>
-      <origin xyz="0 0 1" rpy="0 0 0"/>
-      <mass value="0.0001"/>
-      <inertia
-        ixx="1.0" ixy="0.0" ixz="0.0"
-        iyy="1.0" iyz="0.0"
-        izz="1.0"/>
+      <mass value="0.1" />
+      <origin xyz="0 0 0" rpy="0 0 0"/>
+      <inertia ixx="1" ixy="0" ixz="0" iyy="1" iyz="0" izz="1" />
     </inertial>
     <visual>
@@ -235,17 +220,14 @@
       lower="0"
       upper="3.141"
-      effort="0"
-      velocity="0.01" />
-   <dynamics damping="0.0" friction="0.0" />
+      effort="10000"
+      velocity="0.01" />
+   <dynamics damping="10.0" friction="10.0" />
   </joint>
   <link
     name="finger_2_med_link">
     <inertial>
-      <origin xyz="0 0 1" rpy="0 0 0"/>
-      <mass value="0.0001"/>
-      <inertia
-        ixx="1.0" ixy="0.0" ixz="0.0"
-        iyy="1.0" iyz="0.0"
-        izz="1.0"/>
+      <mass value="0.1" />
+      <origin xyz="0 0 0" rpy="0 0 0"/>
+      <inertia ixx="1" ixy="0" ixz="0" iyy="1" iyz="0" izz="1" />
     </inertial>
     <visual>
@@ -288,17 +270,14 @@
       lower="0.0"
       upper="2.44"
-      effort="0"
-      velocity="0.01" />
-   <dynamics damping="0.0" friction="0.0" />
+      effort="10000"
+      velocity="0.01" />
+   <dynamics damping="10.0" friction="10.0" />
   </joint>
   <link
     name="finger_2_dist_link">
     <inertial>
-      <origin xyz="0 0 1" rpy="0 0 0"/>
-      <mass value="0.0001"/>
-      <inertia
-        ixx="1.0" ixy="0.0" ixz="0.0"
-        iyy="1.0" iyz="0.0"
-        izz="1.0"/>
+      <mass value="0.001" />
+      <origin xyz="0 0 0" rpy="0 0 0"/>
+      <inertia ixx="1" ixy="0" ixz="0" iyy="1" iyz="0" izz="1" />
     </inertial>
     <visual>
@@ -341,17 +320,14 @@
       lower="0.6"
       upper="1.57"
-      effort="0"
-      velocity="0.01" />
-   <dynamics damping="0.0" friction="0.0" />
+      effort="10000"
+      velocity="0.01" />
+   <dynamics damping="10.0" friction="10.0" />
   </joint>
   <link
     name="finger_3_med_link">
     <inertial>
-      <origin xyz="0 0 1" rpy="0 0 0"/>
-      <mass value="0.0001"/>
-      <inertia
-        ixx="1.0" ixy="0.0" ixz="0.0"
-        iyy="1.0" iyz="0.0"
-        izz="1.0"/>
+      <mass value="0.1" />
+      <origin xyz="-0.05 0 0" rpy="0 0 0"/>
+      <inertia ixx="1.0" ixy="0" ixz="0" iyy="1.0" iyz="0" izz="1.0" />
     </inertial>
     <visual>
@@ -394,17 +370,14 @@
       lower="0.0"
       upper="2.44"
-      effort="0"
-      velocity="0.01" />
-   <dynamics damping="0.0" friction="0.0" />
+      effort="10000"
+      velocity="0.01" />
+   <dynamics damping="1.0" friction="1000.0" />
   </joint>
   <link
     name="finger_3_dist_link">
     <inertial>
-      <origin xyz="0 0 1" rpy="0 0 0"/>
-      <mass value="0.0001"/>
-      <inertia
-        ixx="1.0" ixy="0.0" ixz="0.0"
-        iyy="1.0" iyz="0.0"
-        izz="1.0"/>
+      <mass value="0.1" />
+      <origin xyz="-0.04 0 0" rpy="0 0 0"/>
+      <inertia ixx="1.0" ixy="0" ixz="0" iyy="1.0" iyz="0" izz="1.0" />
     </inertial>
     <visual>
@@ -447,7 +420,7 @@
       lower="0.6"
       upper="1.57"
-      effort="0"
+      effort="10000"
       velocity="0" />
-   <dynamics damping="0.0" friction="0.0" />
+   <dynamics damping="10.0" friction="10.0" />
   </joint>
   <transmission name="tran11">

Commit message: barrett hand tip joints are now underactuaded in URDF

File: barrett_hand_description/urdf/barrett_hand.xacro (robot description, xacro)
@@ -1,4 +1,6 @@
 <?xml version="1.0"?>
 <robot xmlns:xacro="http://www.ros.org/wiki/xacro">
+  <property name="dist_joint_offset" value="0.75" />
+  <property name="dist_joint_multiplier" value="0.3" />
   <link name="barrett_base_link">
     <inertial>
@@ -173,4 +175,5 @@
       velocity="0.01" />
    <dynamics damping="10.0" friction="10.0" />
+   <mimic joint="finger_1_med_joint" multiplier="${dist_joint_multiplier}" offset="${dist_joint_offset}"/>
   </joint>
   <link
@@ -323,4 +326,5 @@
       velocity="0.01" />
    <dynamics damping="10.0" friction="10.0" />
+   <mimic joint="finger_2_med_joint" multiplier="${dist_joint_multiplier}" offset="${dist_joint_offset}"/>
   </joint>
   <link
@@ -423,4 +427,5 @@
       velocity="0" />
    <dynamics damping="10.0" friction="10.0" />
+   <mimic joint="finger_3_med_joint" multiplier="${dist_joint_multiplier}" offset="${dist_joint_offset}"/>
   </joint>
   <transmission name="tran11">

Commit message: Barrett hand working in gazebo!

File: barrett_hand_description/urdf/barrett_hand.xacro (robot description, xacro)
@@ -27,4 +27,11 @@
     </collision>
   </link>
+  <joint name="palm_joint" type="fixed"> <!--original is revolute-->
+    <origin xyz="0.0 0.0 0.077"/>
+    <parent link="barrett_base_link" />
+    <child link="palm_frame" />
+  </joint>
+  <link name="palm_frame">
+  </link>
   <link name="finger_1_prox_link">
     <inertial>
@@ -57,21 +64,10 @@
     </collision>
   </link>
-  <joint
-    name="finger_1_prox_joint"
-    type="revolute">
-    <origin
-      xyz="0.025 0 0.0415"
-      rpy="0 2.7051E-17 -1.5708" />
-    <parent
-      link="barrett_base_link" />
-    <child
-      link="finger_1_prox_link" />
-    <axis
-      xyz="0 0 -1" />
-    <limit
-      lower="0.0"
-      upper="3.141"
-      effort="10000"
-      velocity="0.01" />
+  <joint name="finger_1_prox_joint" type="revolute">
+    <origin xyz="0.025 0 0.0415" rpy="0 2.7051E-17 -1.5708" />
+    <parent link="barrett_base_link" />
+    <child link="finger_1_prox_link" />
+    <axis xyz="0 0 -1" />
+    <limit lower="0.0" upper="3.141" effort="10000" velocity="0.2" />
    <dynamics damping="10.0" friction="10.0" />
   </joint>
@@ -110,18 +106,9 @@
     name="finger_1_med_joint"
     type="revolute">
-    <origin
-      xyz="-0.05 0 0.0339"
-      rpy="-1.5708 -8.8281E-17 0" />
-    <parent
-      link="finger_1_prox_link" />
-    <child
-      link="finger_1_med_link" />
-    <axis
-      xyz="0 0 1" />
-    <limit
-      lower="0"
-      upper="2.44"
-      effort="10000"
-      velocity="0.01" />
+    <origin xyz="-0.05 0 0.0339" rpy="-1.5708 -8.8281E-17 0" />
+    <parent link="finger_1_prox_link" />
+    <child link="finger_1_med_link" />
+    <axis xyz="0 0 1" />
+    <limit lower="0" upper="2.44" effort="10000" velocity="0.2" />
    <dynamics damping="10.0" friction="10.0" />
   </joint>
@@ -134,44 +121,25 @@
     </inertial>
     <visual>
-      <origin
-        xyz="0 0 0"
-        rpy="3.14159265359 0 -0.73" />
-      <geometry>
-        <mesh
-          filename="package://barrett_hand_description/meshes/finger_1_dist_link.STL" />
-      </geometry>
-      <material
-        name="">
-        <color
-          rgba="0.898039215686275 0.917647058823529 0.929411764705882 1" />
-      </material>
-    </visual>
-    <collision>
-      <origin
-        xyz="0 0 0"
-        rpy="3.14159265359 0 -0.73" />
-      <geometry>
-        <mesh
-          filename="package://barrett_hand_description/meshes/finger_1_dist_link.STL" />
-      </geometry>
-    </collision>
-  </link>
-  <joint
-    name="finger_1_dist_joint"
-    type="revolute"> <!--original is revolute-->
-    <origin
-      xyz="-0.069936 -0.003 0"
-      rpy="1.6787E-18 -3.6382E-15 -6.1073E-33" />
-    <parent
-      link="finger_1_med_link" />
-    <child
-      link="finger_1_dist_link" />
-    <axis
-      xyz="0 0 1" />
-    <limit
-      lower="0.6"
-      upper="1.57"
-      effort="10000"
-      velocity="0.01" />
+      <origin xyz="0 0 0" rpy="3.14159265359 0 -0.73" />
+      <geometry>
+        <mesh filename="package://barrett_hand_description/meshes/finger_1_dist_link.STL" />
+      </geometry>
+      <material name="">
+        <color rgba="0.898039215686275 0.917647058823529 0.929411764705882 1" />
+      </material>
+    </visual>
+    <collision>
+      <origin xyz="0 0 0" rpy="3.14159265359 0 -0.73" />
+      <geometry>
+        <mesh filename="package://barrett_hand_description/meshes/finger_1_dist_link.STL" />
+      </geometry>
+    </collision>
+  </link>
+  <joint name="finger_1_dist_joint" type="revolute"> <!--original is revolute-->
+    <origin xyz="-0.069936 -0.003 0" rpy="1.6787E-18 -3.6382E-15 -6.1073E-33" />
+    <parent link="finger_1_med_link" />
+    <child link="finger_1_dist_link" />
+    <axis xyz="0 0 1" />
+    <limit lower="0.6" upper="1.57" effort="10000" velocity="0.2" />
    <dynamics damping="10.0" friction="10.0" />
    <mimic joint="finger_1_med_joint" multiplier="${dist_joint_multiplier}" offset="${dist_joint_offset}"/>
@@ -185,10 +153,41 @@
     </inertial>
     <visual>
-      <origin
-        xyz="0 0 0"
-        rpy="0 0 0" />
-      <geometry>
-        <mesh
-          filename="package://barrett_hand_description/meshes/finger_2_prox_link.STL" />
+      <origin xyz="0 0 0" rpy="0 0 0" />
+      <geometry>
+        <mesh filename="package://barrett_hand_description/meshes/finger_2_prox_link.STL" />
+      </geometry>
+      <material name="">
+        <color rgba="0.752941176470588 0.752941176470588 0.752941176470588 1" />
+      </material>
+    </visual>
+    <collision>
+      <origin xyz="0 0 0" rpy="0 0 0" />
+      <geometry>
+        <mesh filename="package://barrett_hand_description/meshes/finger_2_prox_link.STL" />
+      </geometry>
+    </collision>
+  </link>
+  <joint name="finger_2_prox_joint" type="revolute">
+    <origin xyz="-0.025 0 0.0415" rpy="0 2.7051E-17 -1.5708" />
+    <parent link="barrett_base_link" />
+    <child link="finger_2_prox_link" />
+    <axis xyz="0 0 1" />
+    <limit lower="0" upper="3.141" effort="10000"  velocity="0.2" />
+   <dynamics damping="10.0" friction="10.0" />
+  </joint>
+  <link
+    name="finger_2_med_link">
+    <inertial>
+      <mass value="0.1" />
+      <origin xyz="0 0 0" rpy="0 0 0"/>
+      <inertia ixx="1" ixy="0" ixz="0" iyy="1" iyz="0" izz="1" />
+    </inertial>
+    <visual>
+      <origin
+        xyz="0 0 0"
+        rpy="3.14159265359 0 0" />
+      <geometry>
+        <mesh
+          filename="package://barrett_hand_description/meshes/finger_2_med_link.STL" />
       </geometry>
       <material
@@ -201,54 +200,4 @@
       <origin
         xyz="0 0 0"
-        rpy="0 0 0" />
-      <geometry>
-        <mesh
-          filename="package://barrett_hand_description/meshes/finger_2_prox_link.STL" />
-      </geometry>
-    </collision>
-  </link>
-  <joint
-    name="finger_2_prox_joint"
-    type="revolute">
-    <origin
-      xyz="-0.025 0 0.0415"
-      rpy="0 2.7051E-17 -1.5708" />
-    <parent
-      link="barrett_base_link" />
-    <child
-      link="finger_2_prox_link" />
-    <axis
-      xyz="0 0 1" />
-    <limit
-      lower="0"
-      upper="3.141"
-      effort="10000"
-      velocity="0.01" />
-   <dynamics damping="10.0" friction="10.0" />
-  </joint>
-  <link
-    name="finger_2_med_link">
-    <inertial>
-      <mass value="0.1" />
-      <origin xyz="0 0 0" rpy="0 0 0"/>
-      <inertia ixx="1" ixy="0" ixz="0" iyy="1" iyz="0" izz="1" />
-    </inertial>
-    <visual>
-      <origin
-        xyz="0 0 0"
-        rpy="3.14159265359 0 0" />
-      <geometry>
-        <mesh
-          filename="package://barrett_hand_description/meshes/finger_2_med_link.STL" />
-      </geometry>
-      <material
-        name="">
-        <color
-          rgba="0.752941176470588 0.752941176470588 0.752941176470588 1" />
-      </material>
-    </visual>
-    <collision>
-      <origin
-        xyz="0 0 0"
         rpy="3.14159265359 0 0" />
       <geometry>
@@ -261,18 +210,9 @@
     name="finger_2_med_joint"
     type="revolute">
-    <origin
-      xyz="-0.05 0 0.0339"
-      rpy="-1.5708 -8.8281E-17 0" />
-    <parent
-      link="finger_2_prox_link" />
-    <child
-      link="finger_2_med_link" />
-    <axis
-      xyz="0 0 1" />
-    <limit
-      lower="0.0"
-      upper="2.44"
-      effort="10000"
-      velocity="0.01" />
+    <origin xyz="-0.05 0 0.0339" rpy="-1.5708 -8.8281E-17 0" />
+    <parent link="finger_2_prox_link" />
+    <child link="finger_2_med_link" />
+    <axis xyz="0 0 1" />
+    <limit lower="0.0" upper="2.44" effort="10000" velocity="0.2" />
    <dynamics damping="10.0" friction="10.0" />
   </joint>
@@ -285,15 +225,10 @@
     </inertial>
     <visual>
-      <origin
-        xyz="0 0 0"
-        rpy="3.14159265359 0 -0.73" />
-      <geometry>
-        <mesh
-          filename="package://barrett_hand_description/meshes/finger_2_dist_link.STL" />
-      </geometry>
-      <material
-        name="">
-        <color
-          rgba="0.898039215686275 0.917647058823529 0.929411764705882 1" />
+      <origin xyz="0 0 0" rpy="3.14159265359 0 -0.73" />
+      <geometry>
+        <mesh filename="package://barrett_hand_description/meshes/finger_2_dist_link.STL" />
+      </geometry>
+      <material name="">
+        <color rgba="0.898039215686275 0.917647058823529 0.929411764705882 1" />
       </material>
     </visual>
@@ -324,5 +259,5 @@
       upper="1.57"
       effort="10000"
-      velocity="0.01" />
+      velocity="0.2" />
    <dynamics damping="10.0" friction="10.0" />
    <mimic joint="finger_2_med_joint" multiplier="${dist_joint_multiplier}" offset="${dist_joint_offset}"/>
@@ -375,6 +310,6 @@
       upper="2.44"
       effort="10000"
-      velocity="0.01" />
-   <dynamics damping="1.0" friction="1000.0" />
+      velocity="0.2" />
+   <dynamics damping="10.0" friction="10.0" />
   </joint>
   <link
@@ -425,5 +360,5 @@
       upper="1.57"
       effort="10000"
-      velocity="0" />
+      velocity="0.2" />
    <dynamics damping="10.0" friction="10.0" />
    <mimic joint="finger_3_med_joint" multiplier="${dist_joint_multiplier}" offset="${dist_joint_offset}"/>
@@ -442,5 +377,5 @@
     <actuator name="motor12">
       <hardwareInterface>EffortJointInterface</hardwareInterface>
-      <mechanicalReduction>10</mechanicalReduction>
+      <mechanicalReduction>1</mechanicalReduction>
     </actuator>
   </transmission>
