Commit message: - added missing joint defs

File: barrett_hand_description/urdf/barrett_hand.xacro (robot description, xacro)
@@ -366,5 +366,7 @@
   <transmission name="tran11">
     <type>transmission_interface/SimpleTransmission</type>
-    <joint name="finger_1_med_joint"/>
+    <joint name="finger_1_med_joint">
+        <hardwareInterface>PositionJointInterface</hardwareInterface>
+    </joint>
     <actuator name="motor11">
       <hardwareInterface>EffortJointInterface</hardwareInterface>
@@ -374,5 +376,7 @@
   <transmission name="tran12">
     <type>transmission_interface/SimpleTransmission</type>
-    <joint name="finger_1_dist_joint"/>
+    <joint name="finger_1_dist_joint">
+      <hardwareInterface>PositionJointInterface</hardwareInterface>
+    </joint>
     <actuator name="motor12">
       <hardwareInterface>EffortJointInterface</hardwareInterface>
@@ -382,5 +386,7 @@
   <transmission name="tran13">
     <type>transmission_interface/SimpleTransmission</type>
-    <joint name="finger_2_med_joint"/>
+    <joint name="finger_2_med_joint">
+      <hardwareInterface>PositionJointInterface</hardwareInterface>
+    </joint>
     <actuator name="motor13">
       <hardwareInterface>EffortJointInterface</hardwareInterface>
@@ -390,5 +396,7 @@
   <transmission name="tran14">
     <type>transmission_interface/SimpleTransmission</type>
-    <joint name="finger_2_dist_joint"/>
+    <joint name="finger_2_dist_joint">
+      <hardwareInterface>PositionJointInterface</hardwareInterface>
+    </joint>
     <actuator name="motor14">
       <hardwareInterface>EffortJointInterface</hardwareInterface>
@@ -398,5 +406,7 @@
   <transmission name="tran15">
     <type>transmission_interface/SimpleTransmission</type>
-    <joint name="finger_3_med_joint"/>
+    <joint name="finger_3_med_joint">
+      <hardwareInterface>PositionJointInterface</hardwareInterface>
+    </joint>
     <actuator name="motor15">
       <hardwareInterface>EffortJointInterface</hardwareInterface>
@@ -406,5 +416,7 @@
   <transmission name="tran16">
     <type>transmission_interface/SimpleTransmission</type>
-    <joint name="finger_3_dist_joint"/>
+    <joint name="finger_3_dist_joint">
+      <hardwareInterface>PositionJointInterface</hardwareInterface>
+    </joint>
     <actuator name="motor16">
       <hardwareInterface>EffortJointInterface</hardwareInterface>
@@ -414,5 +426,7 @@
   <transmission name="tran17">
     <type>transmission_interface/SimpleTransmission</type>
-    <joint name="finger_1_prox_joint"/>
+    <joint name="finger_1_prox_joint">
+      <hardwareInterface>PositionJointInterface</hardwareInterface>
+    </joint>
     <actuator name="motor17">
       <hardwareInterface>EffortJointInterface</hardwareInterface>
@@ -422,5 +436,7 @@
   <transmission name="tran18">
     <type>transmission_interface/SimpleTransmission</type>
-    <joint name="finger_2_prox_joint"/>
+    <joint name="finger_2_prox_joint">
+      <hardwareInterface>PositionJointInterface</hardwareInterface>
+    </joint>
     <actuator name="motor18">
       <hardwareInterface>EffortJointInterface</hardwareInterface>
